File: PCB/Quantum-SAX.kicad_pcb (KiCad board)
At the start: 2 copper layers, 287.5 x 132.4 mm, 62 parts, among them J1 USB C Connector, J2 JTAG_TC2030, SW1 Boot, U1 XC6206, U2 USBLC6-2SC6, U3 RP2040, U4 W25Q128JVS, Y1 12MHz

Commit message: Finished routing
Parts:
- added G***: LOGO, LOGO, B.Cu at (193.8, 96.3)
- added H1: qw-logo, qw-logo:qw new logo silk + copper md, F.Cu at (60.1, 59.9)
- added H2: qw-logo, qw-logo:qw new logo silk + copper sm, B.Cu at (255.6, 60.0)
- added H3: 1999-logo, 1999:1999 logo md, F.Cu at (57.9, 170.9)
- added H4: 1999-logo, 1999:1999 logo md, B.Cu at (74.9, 78.6)
- R4: value 470 -> 10k
- moved C15 0.62 mm to (187.8, 80.5)
Connections:
- CH1 pad 1: unconnected-(CH1-Pad1) -> GND
- CH1 pad 2: unconnected-(CH1-Pad2) -> START
- CH10 pad 1: unconnected-(CH10-Pad1) -> GND
- CH10 pad 2: unconnected-(CH10-Pad2) -> C_DN
- CH11 pad 1: unconnected-(CH11-Pad1) -> GND
- CH11 pad 2: unconnected-(CH11-Pad2) -> A
- CH12 pad 1: unconnected-(CH12-Pad1) -> GND
- CH12 pad 2: unconnected-(CH12-Pad2) -> C_RT
- CH13 pad 1: unconnected-(CH13-Pad1) -> GND
- CH13 pad 2: unconnected-(CH13-Pad2) -> C_LT
- CH14 pad 1: unconnected-(CH14-Pad1) -> GND
- CH14 pad 2: unconnected-(CH14-Pad2) -> C_UP
- CH15 pad 1: unconnected-(CH15-Pad1) -> GND
- CH15 pad 2: unconnected-(CH15-Pad2) -> B
- CH16 pad 1: unconnected-(CH16-Pad1) -> GND
- CH16 pad 2: unconnected-(CH16-Pad2) -> X
- CH17 pad 1: unconnected-(CH17-Pad1) -> GND
- CH17 pad 2: unconnected-(CH17-Pad2) -> Z
- CH18 pad 1: unconnected-(CH18-Pad1) -> GND
- CH18 pad 2: unconnected-(CH18-Pad2) -> UP
- CH19 pad 1: unconnected-(CH19-Pad1) -> GND
- CH19 pad 2: unconnected-(CH19-Pad2) -> R
- CH2 pad 1: unconnected-(CH2-Pad1) -> GND
- CH2 pad 2: unconnected-(CH2-Pad2) -> L
- CH20 pad 1: unconnected-(CH20-Pad1) -> GND
- CH20 pad 2: unconnected-(CH20-Pad2) -> Y
- CH21 pad 1: unconnected-(CH21-Pad1) -> GND
- CH21 pad 2: unconnected-(CH21-Pad2) -> LS
- CH22 pad 1: unconnected-(CH22-Pad1) -> GND
- CH22 pad 2: unconnected-(CH22-Pad2) -> MS
- CH3 pad 1: unconnected-(CH3-Pad1) -> GND
- CH3 pad 2: unconnected-(CH3-Pad2) -> LEFT
- CH4 pad 1: unconnected-(CH4-Pad1) -> GND
- CH4 pad 2: unconnected-(CH4-Pad2) -> DOWN
- CH5 pad 1: unconnected-(CH5-Pad1) -> GND
- CH5 pad 2: unconnected-(CH5-Pad2) -> RIGHT
- CH6 pad 1: unconnected-(CH6-Pad1) -> GND
- CH6 pad 2: unconnected-(CH6-Pad2) -> UP2
- CH7 pad 1: unconnected-(CH7-Pad1) -> GND
- CH7 pad 2: unconnected-(CH7-Pad2) -> M1
- CH8 pad 1: unconnected-(CH8-Pad1) -> GND
- CH8 pad 2: unconnected-(CH8-Pad2) -> M2
- CH9 pad 1: unconnected-(CH9-Pad1) -> GND
- CH9 pad 2: unconnected-(CH9-Pad2) -> M3
- U3 pad 11: unconnected-(U3-GPIO8-Pad11) -> M3
- U3 pad 3: unconnected-(U3-GPIO1-Pad3) -> UP2
Routing:
- net C_DN: track 15.1 -> 186.8 mm
- net MS: track 15.9 -> 187.0 mm
- net L: track 17.3 -> 175.0 mm
- net LS: track 14.8 -> 170.6 mm
- net UP: track 16.4 -> 171.5 mm
- net C_LT: track 16.5 -> 161.1 mm
- net LEFT: track 17.3 -> 160.6 mm
- net Z: track 15.9 -> 153.0 mm
- net A: track 16.0 -> 149.4 mm
- net Y: track 15.5 -> 142.3 mm
- net DOWN: track 16.9 -> 131.4 mm
- net M2: track 18.6 -> 128.0 mm
- net X: track 14.9 -> 124.1 mm
- net C_UP: track 17.3 -> 123.6 mm
- net M3: track 0.00 -> 103.3 mm
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Other:
- board text added: "Quantum-SAX by Quark quark.works"
- board text added: "S A X"
- board text added: "quark.works"

Commit message: Production files and case files
Parts:
- added H10: MountingHole, MountingHole:MountingHole_2.2mm_M2, F.Cu at (254.8, 155.1)
- added H11: MountingHole, MountingHole:MountingHole_2.2mm_M2, F.Cu at (119.2, 111.8)
- added H12: MountingHole, MountingHole:MountingHole_2.2mm_M2, F.Cu at (171.8, 53.8)
- added H13: MountingHole, MountingHole:MountingHole_2.2mm_M2, F.Cu at (211.8, 53.8)
- added H14: MountingHole, MountingHole:MountingHole_2.2mm_M2, F.Cu at (307.6, 100.0)
- added H15: MountingHole, MountingHole:MountingHole_2.2mm_M2, F.Cu at (71.8, 163.8)
- added H16: MountingHole, MountingHole:MountingHole_2.2mm_M2, F.Cu at (311.8, 163.8)
- added H5: MountingHole, MountingHole:MountingHole_2.2mm_M2, F.Cu at (103.0, 70.0)
- added H6: MountingHole, MountingHole:MountingHole_2.2mm_M2, F.Cu at (156.0, 137.7)
- added H7: MountingHole, MountingHole:MountingHole_2.2mm_M2, F.Cu at (193.7, 160.5)
- added H8: MountingHole, MountingHole:MountingHole_2.2mm_M2, F.Cu at (285.3, 70.5)
- added H9: MountingHole, MountingHole:MountingHole_2.2mm_M2, F.Cu at (215.1, 126.8)
- moved H2 59.0 mm to (314.6, 60.6)
Routing:
- net UP: track 171.5 -> 170.0 mm
Other:
- board text added: "Quantum-SAX by Quark quark.works 19.99"
- board text removed: "Quantum-SAX by Quark quark.works"
