File: PCB/Quantum-SAX.kicad_sch (KiCad schematic)
At the start: 62 parts, among them J1 USB C Connector, J2 JTAG_TC2030, SW1 Boot, U1 XC6206, U2 USBLC6-2SC6, U3 RP2040, U4 W25Q128JVS, Y1 12MHz

Commit message: Finished routing
Parts:
- added H1: qw-logo, qw-logo:qw new logo silk + copper md, symbol Mechanical:MountingHole
- added H2: qw-logo, qw-logo:qw new logo silk + copper sm, symbol Mechanical:MountingHole
- added H3, H4: 1999-logo, 1999:1999 logo md, symbol Mechanical:MountingHole
- R4: value 470 -> 10k
Connections:
- net A: now also CH11.2
- net B: now also CH15.2
- net C_DN: now also CH10.2
- net C_LT: now also CH13.2
- net C_RT: now also CH12.2
- net C_UP: now also CH14.2
- net DOWN: now also CH4.2
- net GND: now also CH1.1, CH10.1, CH11.1, CH12.1, CH13.1, CH14.1, CH15.1, CH16.1, CH17.1, CH18.1, CH19.1, CH2.1, CH20.1, CH21.1, CH22.1, CH3.1, CH4.1, CH5.1, CH6.1, CH7.1, CH8.1, CH9.1
- net L: now also CH2.2
- net LEFT: now also CH3.2
- net LS: now also CH21.2
- net M1: now also CH7.2
- net M2: now also CH8.2
- net MS: now also CH22.2
- net R: now also CH19.2
- net RIGHT: now also CH5.2
- net START: now also CH1.2
- net UP: now also CH18.2
- net X: now also CH16.2
- net Y: now also CH20.2
- net Z: now also CH17.2
- net M3: now reaches CH9.2
- net M3: now also U3.11 (GPIO8)
- net UP2: now reaches U3.3 (GPIO1)
- net UP2: now also CH6.2
- no-connect marks 11 -> 10
Other:
- moved on the sheet: CH1, CH10, CH11, CH12, CH13, CH14, CH15, CH16, CH17, CH18, CH19, CH2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

Commit message: Production files and case files
Parts:
- added H10, H11, H12, H13, H14, H15, H16, H5, H6, H7, H8, H9: MountingHole, MountingHole:MountingHole_2.2mm_M2, symbol Mechanical:MountingHole
- D1, D2: LCSC C130880 -> C8598
- SW1: now in the parts list
